File: pcb/Fabricate_Wireless_Macropad.kicad_pcb (KiCad board)
At the start: 2 copper layers, 84 x 78 mm, 71 parts, among them J1 PROTECTED_1S_LIPO_3.7V, Q1 AO3401A, Q2 AO3401A, SW1 MX_KEY_1, SW2 MX_KEY_2, SW3 MX_KEY_3, SW4 MX_KEY_4, SW5 MX_KEY_5, SW6 MX_KEY_6, SW7 JS102011SAQN, U1 XIAO_ESP32S3, U2 MCP23008-xP, U3 TPS61023DRL, U4 74AHCT1G125

Commit message: Updated wih cheeaper pads
Parts:
- added JP1: MODE_SELECT, Jumper:SolderJumper-3_P1.3mm_Open_Pad1.0x1.5mm, B.Cu at (64.0, 98.0)
- added JP2: MODE_SELECT, Jumper:SolderJumper-2_P1.3mm_Open_Pad1.0x1.5mm, B.Cu at (64.0, 124.0)
- added JP3: MODE_SELECT, Jumper:SolderJumper-2_P1.3mm_Open_Pad1.0x1.5mm, B.Cu at (113.0, 94.0)
- added JP4: MODE_SELECT, Jumper:SolderJumper-3_P1.3mm_Open_Pad1.0x1.5mm, B.Cu at (64.0, 128.0)
- added JP5: MODE_SELECT, Jumper:SolderJumper-3_P1.3mm_Open_Pad1.0x1.5mm, B.Cu at (64.0, 135.0)
- added JP6: MODE_SELECT, Jumper:SolderJumper-2_P1.3mm_Open_Pad1.0x1.5mm, B.Cu at (65.0, 74.0)
- added JP7: MODE_SELECT, Jumper:SolderJumper-2_P1.3mm_Open_Pad1.0x1.5mm, B.Cu at (68.0, 70.0)
- U2: value MCP23008-xP -> MCP23008-E/SO; footprint Package_DIP:DIP-18_W7.62mm -> Package_SO:SOIC-18W_7.5x11.6mm_P1.27mm
- moved U2 10.8 mm to (57.2, 110.2), turned to 0 degrees
Connections:
- U1 pad 1: RGB_EN -> MCU_D0
- U1 pad 3: unconnected-(U1-D2_GPIO3-Pad3) -> MCU_D2
- U1 pad 4: unconnected-(U1-D3_GPIO4-Pad4) -> MCU_D3
- U1 pad 5: SDA -> MCU_D4
- U1 pad 6: SCL -> MCU_D5
- U1 pad 7: unconnected-(U1-D6_GPIO43-Pad7) -> MCU_D6
Routing:
- net MCU_D2: track 0.00 -> 123.0 mm, vias 0 -> 2
- net MCU_D5: track 0.00 -> 83.0 mm, vias 0 -> 2
- net MCU_D4: track 0.00 -> 74.1 mm, vias 0 -> 3
- net GND: track 426.0 -> 368.6 mm, vias 9 -> 24
- net MCU_D3: track 0.00 -> 49.7 mm, vias 0 -> 4
- net COL0: track 42.4 -> 91.1 mm, vias 2 -> 4
- net MCU_D0: track 0.00 -> 43.1 mm, vias 0 -> 3
- net RGB_EN: track 21.4 -> 63.5 mm, vias 0 -> 5
- net SCL: track 41.3 -> 77.6 mm, vias 1 -> 5
- net VBUS: track 17.2 -> 52.4 mm, vias 0 -> 2
- net MCU_D6: track 0.00 -> 33.0 mm, vias 0 -> 1
- net COL3: track 88.5 -> 117.7 mm, vias 1 -> 0
- net +5V_RGB: track 392.7 -> 420.3 mm, vias 8 -> 10
- net ROW1: track 93.6 -> 117.7 mm, vias 1 -> 3
- net COL1: track 71.3 -> 92.1 mm, vias 1 -> 6
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