File: pcb/Fabricate_Wireless_Macropad.kicad_sch (KiCad schematic)
At the start: 26 parts, among them J1 PROTECTED_1S_LIPO_3.7V, Q1 AO3401A, Q2 AO3401A, SW1 MX_KEY_1, SW2 MX_KEY_2, SW3 MX_KEY_3, SW4 MX_KEY_4, SW5 MX_KEY_5, SW6 MX_KEY_6, SW7 JS102011SAQN, U1 XIAO_ESP32S3

Commit message: Updated wih cheeaper pads
Parts:
- R1, R2: now not fitted
Connections:
- net SCL: no longer U1.6 (D5_GPIO6_SCL)
- net SDA: no longer U1.5 (D4_GPIO5_SDA)
- net MCU_D2: now reaches U1.3 (D2_GPIO3)
- net MCU_D3: now reaches U1.4 (D3_GPIO4)
- net MCU_D6: now reaches U1.7 (D6_GPIO43)
- net RGB_EN renamed MCU_D0
- new net MCU_D4: U1.5 (D4_GPIO5_SDA)
- new net MCU_D5: U1.6 (D5_GPIO6_SCL)
- no-connect marks 4 -> 1
Other:
- added sheet Build_Options (Build_Options.kicad_sch)
Changed lines of the file:
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@@
 		(on_board yes)
 		(in_pos_files yes)
-		(dnp no)
+		(dnp yes)
 		(property "Reference" "R1"
 			(at 40.64 152.4 0)
@@
 		(on_board yes)
 		(in_pos_files yes)
-		(dnp no)
+		(dnp yes)
 		(property "Reference" "R2"
 			(at 58.42 152.4 0)
@@
 	(wire
 		(pts
-			(xy 157.48000000000002 48.26) (xy 157.48 57.15)
+			(xy 157.48 48.26)
+			(xy 157.48 57.15)
 		)
 		(stroke
@@
 	(wire
 		(pts
-			(xy 200.66000000000003 48.26) (xy 200.66 57.15)
+			(xy 200.66 48.26)
+			(xy 200.66 57.15)
 		)
 		(stroke
@@
 	(wire
 		(pts
-			(xy 243.84 48.26) (xy 243.84 57.15)
+			(xy 243.84 48.26)
+			(xy 243.84 57.15)
 		)
 		(stroke
@@
 	(wire
 		(pts
-			(xy 157.48000000000002 81.28) (xy 157.48 90.17)
+			(xy 157.48 81.28)
+			(xy 157.48 90.17)
 		)
 		(stroke
@@
 	(wire
 		(pts
-			(xy 200.66000000000003 81.28) (xy 200.66 90.17)
+			(xy 200.66 81.28)
+			(xy 200.66 90.17)
 		)
 		(stroke
@@
 	(wire
 		(pts
-			(xy 243.84 81.28) (xy 243.84 90.17)
+			(xy 243.84 81.28)
+			(xy 243.84 90.17)
 		)
 		(stroke
@@
 		)
 	)
-	(global_label "RGB_EN"
-		(at 55.879999999999995 48.26 180)
+	(global_label "MCU_D0"
+		(at 55.88 48.26 180)
 		(effects
 			(font
@@
 	)
 	(global_label "RGB_DATA"
-		(at 55.879999999999995 53.34 180)
-		(effects
-			(font
-				(size 1.27 1.27)
-			)
-			(justify right)
-		)
-	)
-	(global_label "SDA"
-		(at 55.879999999999995 68.58 180)
-		(effects
-			(font
-				(size 1.27 1.27)
-			)
-			(justify right)
-		)
-	)
-	(global_label "SCL"
-		(at 55.879999999999995 73.66 180)
+		(at 55.88 53.34 180)
+		(effects
+			(font
+				(size 1.27 1.27)
+			)
+			(justify right)
+		)
+	)
+	(global_label "MCU_D4"
+		(at 55.88 68.58 180)
+		(effects
+			(font
+				(size 1.27 1.27)
+			)
+			(justify right)
+		)
+	)
+	(global_label "MCU_D5"
+		(at 55.88 73.66 180)
 		(effects
 			(font
@@
 	)
 	(global_label "COL2"
-		(at 233.67999999999998 48.26 180)
+		(at 233.68 48.26 180)
 		(effects
 			(font
@@
 	)
 	(global_label "COL2"
-		(at 233.67999999999998 81.28 180)
+		(at 233.68 81.28 180)
 		(effects
 			(font
@@
 	)
 	(global_label "ENC1_B"
-		(at 157.48 124.46000000000001 180)
+		(at 157.48 124.46 180)
 		(effects
 			(font
@@
 	)
 	(global_label "COL3"
-		(at 172.72 124.46000000000001 0)
+		(at 172.72 124.46 0)
 		(effects
 			(font
@@
 	)
 	(global_label "ENC2_B"
-		(at 226.06 124.46000000000001 180)
+		(at 226.06 124.46 180)
 		(effects
 			(font
@@
 	)
 	(global_label "COL3"
-		(at 241.3 124.46000000000001 0)
+		(at 241.3 124.46 0)
 		(effects
 			(font
@@
 		)
 	)
-	(no_connect
-		(at 55.879999999999995 58.42)
-	)
-	(no_connect
-		(at 55.879999999999995 63.5)
-	)
-	(no_connect
-		(at 55.879999999999995 78.74)
-	)
 	(sheet
 		(at 139.7 154.94)
@@
 	)
 	(global_label "VBAT_GATE"
-		(at 115.57000000000001 119.38 180)
+		(at 115.57 119.38 180)
 		(effects
 			(font
@@
 	)
 	(global_label "VBAT_SWITCH_SOURCE"
-		(at 123.19000000000001 124.46 270)
+		(at 123.19 124.46 270)
 		(effects
 			(font
@@
 	)
 	(global_label "VBAT_RAW"
-		(at 123.19000000000001 114.3 90)
+		(at 123.19 114.3 90)
 		(effects
 			(font
@@
 	)
 	(global_label "VBAT_GATE"
-		(at 120.65 153.67000000000002 270)
+		(at 120.65 153.67 270)
 		(effects
 			(font
@@
 	)
 	(global_label "VBAT_SWITCH_CTRL"
-		(at 158.75 153.67000000000002 270)
+		(at 158.75 153.67 270)
 		(effects
 			(font
@@
 	)
 	(global_label "GND"
-		(at 76.2 111.75999999999999 0)
+		(at 76.2 111.76 0)
 		(effects
 			(font
@@
 		)
 	)
+	(global_label "MCU_D2"
+		(at 55.88 58.42 180)
+		(effects
+			(font
+				(size 1.27 1.27)
+			)
+			(justify right)
+		)
+	)
+	(global_label "MCU_D3"
+		(at 55.88 63.5 180)
+		(effects
+			(font
+				(size 1.27 1.27)
+			)
+			(justify right)
+		)
+	)
+	(global_label "MCU_D6"
+		(at 55.88 78.74 180)
+		(effects
+			(font
+				(size 1.27 1.27)
+			)
+			(justify right)
+		)
+	)
+	(sheet
+		(at 185.42 180.34)
+		(size 40.64 10.16)
+		(fields_autoplaced yes)
+		(stroke
+			(width 0.0006)
+			(type default)
+		)
+		(fill
+			(color 0 0 0 0.0)
+		)
+		(property "Sheetname" "Build_Options"
+			(at 142.24 179.07 0)
+			(effects
+				(font
+					(size 1.27 1.27)
+				)
+				(justify left bottom)
+			)
+		)
+		(property "Sheetfile" "Build_Options.kicad_sch"
+			(at 142.24 191.77 0)
+			(effects
+				(font
+					(size 1.27 1.27)
+				)
+				(justify left top)
+			)
+		)
+		(instances
+			(project "Fabricate_Wireless_Macropad"
+				(path "/eae26e58-6f77-4657-abf4-2b51d059bce3"
+					(page "5")
+				)
+			)
+		)
+	)
