File: pcb/RGB_Power.kicad_sch (KiCad schematic)
At the start: 14 parts, among them U3 TPS61023DRL, U4 74AHCT1G125

Commit message: Updated wih cheeaper pads
Parts:
- C3, C5, D10, D9, L1, R4, R5, R6, U3: now not fitted
Changed lines of the file:
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@@
 		(on_board yes)
 		(in_pos_files yes)
-		(dnp no)
+		(dnp yes)
 		(property "Reference" "U3"
 			(at 127 50.8 0)
@@
 		(on_board yes)
 		(in_pos_files yes)
-		(dnp no)
+		(dnp yes)
 		(property "Reference" "D9"
 			(at 55.88 43.18 0)
@@
 		(on_board yes)
 		(in_pos_files yes)
-		(dnp no)
+		(dnp yes)
 		(property "Reference" "D10"
 			(at 55.88 71.12 0)
@@
 		(on_board yes)
 		(in_pos_files yes)
-		(dnp no)
+		(dnp yes)
 		(property "Reference" "L1"
 			(at 119.38 29.21 0)
@@
 			)
 		)
-    (property "MPN" "SRP5030T-1R0M" (at 119.38 35.56 0)
-      (effects (font (size 1.27 1.27)) (hide yes))
-    )
-    (property "Manufacturer" "Bourns" (at 119.38 35.56 0)
-      (effects (font (size 1.27 1.27)) (hide yes))
-    )
+		(property "MPN" "SRP5030T-1R0M"
+			(at 119.38 35.56 0)
+			(effects
+				(font
+					(size 1.27 1.27)
+				)
+				(hide yes)
+			)
+		)
+		(property "Manufacturer" "Bourns"
+			(at 119.38 35.56 0)
+			(effects
+				(font
+					(size 1.27 1.27)
+				)
+				(hide yes)
+			)
+		)
 		(pin "1"
 		)
@@
 		(on_board yes)
 		(in_pos_files yes)
-		(dnp no)
+		(dnp yes)
 		(property "Reference" "C3"
 			(at 81.28 63.5 0)
@@
 			)
 		)
-    (property "MPN" "C1206C106K8RACTU" (at 83.82 63.5 0)
-      (effects (font (size 1.27 1.27)) (hide yes))
-    )
-    (property "Manufacturer" "KEMET" (at 83.82 63.5 0)
-      (effects (font (size 1.27 1.27)) (hide yes))
-    )
-    (property "LCSC" "C2167669" (at 83.82 63.5 0)
-      (effects (font (size 1.27 1.27)) (hide yes))
-    )
+		(property "MPN" "C1206C106K8RACTU"
+			(at 83.82 63.5 0)
+			(effects
+				(font
+					(size 1.27 1.27)
+				)
+				(hide yes)
+			)
+		)
+		(property "Manufacturer" "KEMET"
+			(at 83.82 63.5 0)
+			(effects
+				(font
+					(size 1.27 1.27)
+				)
+				(hide yes)
+			)
+		)
+		(property "LCSC" "C2167669"
+			(at 83.82 63.5 0)
+			(effects
+				(font
+					(size 1.27 1.27)
+				)
+				(hide yes)
+			)
+		)
 		(pin "1"
 		)
@@
 			)
 		)
-    (property "MPN" "CL32B226KOJNFNE" (at 170.18 43.18 0)
-      (effects (font (size 1.27 1.27)) (hide yes))
-    )
-    (property "Manufacturer" "Samsung Electro-Mechanics" (at 170.18 43.18 0)
-      (effects (font (size 1.27 1.27)) (hide yes))
-    )
-    (property "LCSC" "C16196563" (at 170.18 43.18 0)
-      (effects (font (size 1.27 1.27)) (hide yes))
-    )
+		(property "MPN" "CL32B226KOJNFNE"
+			(at 170.18 43.18 0)
+			(effects
+				(font
+					(size 1.27 1.27)
+				)
+				(hide yes)
+			)
+		)
+		(property "Manufacturer" "Samsung Electro-Mechanics"
+			(at 170.18 43.18 0)
+			(effects
+				(font
+					(size 1.27 1.27)
+				)
+				(hide yes)
+			)
+		)
+		(property "LCSC" "C16196563"
+			(at 170.18 43.18 0)
+			(effects
+				(font
+					(size 1.27 1.27)
+				)
+				(hide yes)
+			)
+		)
 		(pin "1"
 		)
@@
 		(on_board yes)
 		(in_pos_files yes)
-		(dnp no)
+		(dnp yes)
 		(property "Reference" "C5"
 			(at 205.74 43.18 0)
@@
 			)
 		)
-    (property "MPN" "CL32B226KOJNFNE" (at 208.28 43.18 0)
-      (effects (font (size 1.27 1.27)) (hide yes))
-    )
-    (property "Manufacturer" "Samsung Electro-Mechanics" (at 208.28 43.18 0)
-      (effects (font (size 1.27 1.27)) (hide yes))
-    )
-    (property "LCSC" "C16196563" (at 208.28 43.18 0)
-      (effects (font (size 1.27 1.27)) (hide yes))
-    )
+		(property "MPN" "CL32B226KOJNFNE"
+			(at 208.28 43.18 0)
+			(effects
+				(font
+					(size 1.27 1.27)
+				)
+				(hide yes)
+			)
+		)
+		(property "Manufacturer" "Samsung Electro-Mechanics"
+			(at 208.28 43.18 0)
+			(effects
+				(font
+					(size 1.27 1.27)
+				)
+				(hide yes)
+			)
+		)
+		(property "LCSC" "C16196563"
+			(at 208.28 43.18 0)
+			(effects
+				(font
+					(size 1.27 1.27)
+				)
+				(hide yes)
+			)
+		)
 		(pin "1"
 		)
@@
 		(on_board yes)
 		(in_pos_files yes)
-		(dnp no)
+		(dnp yes)
 		(property "Reference" "R4"
 			(at 175.26 71.12 0)
@@
 		(on_board yes)
 		(in_pos_files yes)
-		(dnp no)
+		(dnp yes)
 		(property "Reference" "R5"
-			(at 213.35999999999999 71.12 0)
+			(at 213.36 71.12 0)
 			(show_name no)
 			(do_not_autoplace no)
@@
 		)
 		(property "Value" "100k_1%"
-			(at 213.35999999999999 75 0)
+			(at 213.36 75 0)
 			(show_name no)
 			(do_not_autoplace no)
@@
 		(on_board yes)
 		(in_pos_files yes)
-		(dnp no)
+		(dnp yes)
 		(property "Reference" "R6"
 			(at 81.28 93.98 0)
@@
 	)
 	(global_label "BOOST_IN"
-		(at 59.690000000000005 45.72 0)
+		(at 59.69 45.72 0)
 		(effects
 			(font
@@
 	)
 	(global_label "BOOST_IN"
-		(at 59.690000000000005 73.66 0)
+		(at 59.69 73.66 0)
 		(effects
 			(font
